Commit message: Updated model with gazebo colors

File: description/robot_core.xacro (robot description, xacro)
@@ -10,4 +10,7 @@
     <material name="blue">
         <color rgba="0 0 1 1" />
+    </material>
+    <material name="red">
+        <color rgba="1 0 0 1" />
     </material>
     <!-- BASE LINK -->
@@ -26,4 +29,5 @@
                 <cylinder radius="0.3" length="0.05"/>
             </geometry>
+            <material name="red"/>
         </visual>
         <collision>
@@ -37,4 +41,9 @@
         </xacro:inertial_cylinder>
     </link>
+    <gazebo reference="chassis">
+        <material>
+            Gazebo/RedGlow
+        </material>
+    </gazebo>
     <!-- LEFT WHEEL LINK -->
     <joint name="left_wheel_joint" type="continuous">
@@ -60,4 +69,9 @@
         </xacro:inertial_cylinder>
     </link>
+    <gazebo reference="left_wheel">
+        <material>
+            Gazebo/Blue
+        </material>
+    </gazebo>
     <!-- RIGHT WHEEL LINK -->
     <joint name="right_wheel_joint" type="continuous">
@@ -83,4 +97,9 @@
         </xacro:inertial_cylinder>
     </link>
+    <gazebo reference="right_wheel">
+        <material>
+            Gazebo/Blue
+        </material>
+    </gazebo>
     <!-- CASTER WHEEL LINK -->
     <joint name="caster_wheel_joint" type="fixed">
@@ -105,3 +124,8 @@
         </xacro:inertial_sphere>
     </link>
+    <gazebo reference="caster_wheel_joint">
+        <material>
+            Gazebo/White
+        </material>
+    </gazebo>
 </robot>
