Commit message: Added Diff Drive control

File: description/robot.urdf.xacro (robot description, xacro)
@@ -2,3 +2,4 @@
 <robot xmlns:xacro="http://www.ros.org/wiki/xacro" name="robot">
     <xacro:include filename="robot_core.xacro" />
+    <xacro:include filename="gazebo_control.xacro" />
 </robot>

File: description/robot_core.xacro (robot description, xacro)
@@ -125,7 +125,7 @@
     </link>
     <gazebo reference="caster_wheel_joint">
-        <material>
-            Gazebo/White
-        </material>
+        <material>Gazebo/White</material>
+        <mu1 value="0.0001"/>
+        <mu2 value="0.0001"/>
     </gazebo>
 </robot>
