Commit message: Set to spawn multiple robots

File: description/gazebo_control.xacro (robot description, xacro)
@@ -3,4 +3,7 @@
     <gazebo>
         <plugin name="diff_drive" filename="libgazebo_ros_diff_drive.so">
+            <ros>
+                <namespace>$(arg namespace)</namespace>
+            </ros>
             <!-- WHEEL Information -->
             <left_joint>left_wheel_joint</left_joint>

File: description/robot_core.xacro (robot description, xacro)
@@ -21,5 +21,5 @@
         <parent link="base_link"/>
         <child link="chassis"/>
-        <origin xyz="0 0 0"/>
+        <origin xyz="$(arg x_pos) 0 0"/>
     </joint>
     <link name="chassis">
@@ -50,5 +50,5 @@
         <parent link="base_link"/>
         <child link="left_wheel"/>
-        <origin xyz="0.0 0.175 0.0" rpy="-${pi/2} 0.0 0.0"/>
+        <origin xyz="$(arg x_pos) 0.175 0.0" rpy="-${pi/2} 0.0 0.0"/>
         <axis xyz="0.0 0.0 1.0"/>
     </joint>
@@ -78,5 +78,5 @@
         <parent link="base_link"/>
         <child link="right_wheel"/>
-        <origin xyz="0.0 -0.175 0.0" rpy="${pi/2} 0.0 0.0"/>
+        <origin xyz="$(arg x_pos) -0.175 0.0" rpy="${pi/2} 0.0 0.0"/>
         <axis xyz="0.0 0.0 -1.0"/>
     </joint>

Commit message: Corrected angle and maximum values

File: description/gazebo_control.xacro (robot description, xacro)
@@ -20,4 +20,5 @@
             <publish_odom_tf>true</publish_odom_tf>
             <publish_wheel_tf>true</publish_wheel_tf>
+            <updateRate>20</updateRate>
         </plugin>
     </gazebo>

File: description/robot_core.xacro (robot description, xacro)
@@ -37,5 +37,5 @@
             </geometry>
         </collision>
-        <xacro:inertial_cylinder mass="1" radius="0.3" length="0.05">
+        <xacro:inertial_cylinder mass="10" radius="0.3" length="0.05">
             <origin xyz="0.0 0.0 0.0" rpy="0.0 0.0 0.0"/>
         </xacro:inertial_cylinder>
@@ -106,5 +106,5 @@
         <parent link="chassis"/>
         <child link="caster_wheel"/>
-        <origin xyz="0.24 0.0 -0.05"/>
+        <origin xyz="0.24 0.0 -0.045"/>
     </joint>
     <link name="caster_wheel">
@@ -129,3 +129,51 @@
         <mu2 value="0.001"/>
     </gazebo>
+     <!-- SECOND CASTER WHEEL LINK -->
+    <joint name="caster_wheel_joint_2nd" type="fixed">
+        <parent link="chassis"/>
+        <child link="caster_wheel_2nd"/>
+        <origin xyz="-0.24 0.0 -0.045"/>
+    </joint>
+    <link name="caster_wheel_2nd">
+        <visual>
+            <geometry>
+                <sphere radius="0.05"/>
+            </geometry>
+            <material name="black"/>
+        </visual>
+        <collision>
+            <geometry>
+                <sphere radius="0.05"/>
+            </geometry>
+        </collision>
+        <xacro:inertial_sphere mass="0.01" radius="0.05">
+            <origin xyz="0.0 0.0 0.0" rpy="0.0 0.0 0.0"/>
+        </xacro:inertial_sphere>
+    </link>
+    <gazebo reference="caster_wheel_joint_2nd">
+        <material>Gazebo/White</material>
+        <mu1 value="0.001"/>
+        <mu2 value="0.001"/>
+    </gazebo>
+    <joint name="front_marker_joint" type="fixed">
+        <parent link="chassis"/>
+        <child link="marker"/>
+        <origin xyz="0.24 0.0 0.05"/>
+    </joint>
+    <link name="marker">
+        <visual>
+            <geometry>
+                <cylinder radius="0.02" length="0.05"/>
+            </geometry>
+            <material name="black"/>
+        </visual>
+        <collision>
+            <geometry>
+                <cylinder radius="0.02" length="0.05"/>
+            </geometry>
+        </collision>
+    </link>
+    <gazebo reference="marker">
+        <material>Gazebo/black</material>
+    </gazebo>
 </robot>

Commit message: Robot goings to target

File: description/gazebo_control.xacro (robot description, xacro)
@@ -5,4 +5,5 @@
             <ros>
                 <namespace>$(arg namespace)</namespace>
+                <remapping>/tf:=/$(arg namespace)/tf</remapping>
             </ros>
             <!-- WHEEL Information -->
@@ -12,6 +13,6 @@
             <wheel_diameter>0.1</wheel_diameter>
             <!-- Limits -->
-            <max_wheel_torque>200</max_wheel_torque>
-            <max_wheel_acceleration>200</max_wheel_acceleration>
+            <max_wheel_torque>1</max_wheel_torque>
+            <max_wheel_acceleration>2</max_wheel_acceleration>
             <!-- Odometry Frame -->
             <odometry_frame>odom</odometry_frame>

File: description/robot_core.xacro (robot description, xacro)
@@ -37,5 +37,5 @@
             </geometry>
         </collision>
-        <xacro:inertial_cylinder mass="10" radius="0.3" length="0.05">
+        <xacro:inertial_cylinder mass="0.3" radius="0.3" length="0.05">
             <origin xyz="0.0 0.0 0.0" rpy="0.0 0.0 0.0"/>
         </xacro:inertial_cylinder>

File: description/target.xacro (robot description, xacro)
@@ -8,5 +8,5 @@
         <parent link="base_link"/>
         <child link="circle"/>
-        <origin xyz="0 1 0"/>
+        <origin xyz="8.0 5.0 0"/>
     </joint>
     <link name="circle">
